File: Simpino_bareminimum/Simpino_bareminimum.kicad_pcb (KiCad board)
At the start: 2 copper layers, 50 x 49.8 mm, 21 parts, among them J1 Conn_01x06_Male, J2 Conn_01x08_Male, J3 Conn_01x08_Male, J4 Conn_01x08_Male, J5 Conn_01x01_Male, SW1 SW_Push, U1 ATmega328P-AU, Y1 16mhz

Commit message: update
Parts:
- moved C1 9.58 mm to (60.2, 63.3), turned to 0 degrees
- moved J5 4.66 mm to (62.1, 70.9)
- moved Y1 1.63 mm to (40.7, 54.5), turned to 90 degrees
Routing:
- net GND: track 76.3 -> 64.2 mm
- net Net-(C4-Pad2): track 71.1 -> 76.3 mm
- net /VCC: track 174.0 -> 179.1 mm
- net Net-(U1-Pad7): track 10.0 -> 5.86 mm
- net Net-(U1-Pad8): track 7.05 -> 6.52 mm

Commit message: update
Parts:
- removed J5: Conn_01x01_Male, Connector_PinHeader_2.54mm:PinHeader_1x01_P2.54mm_Horizontal
- J2: footprint Connector_PinHeader_2.54mm:PinHeader_1x08_P2.54mm_Horizontal -> Connector_PinHeader_2.54mm:PinHeader_1x09_P2.54mm_Horizontal
- moved J2 2.50 mm to (61.5, 71.0)
- moved R5 1.14 mm to (51.8, 30.1), turned to 90 degrees
Connections:
- C4 pad 2: Net-(C4-Pad2) -> /RST
- J2 pad 1: /VCC -> /RST
- J2 pad 2: GND -> /VCC
- J2 pad 3: /D13_SCK -> GND
- J2 pad 4: /D12_MISO -> /D13_SCK
- J2 pad 5: /D11_MOSI -> /D12_MISO
- J2 pad 6: /D10_SS -> /D11_MOSI
- J2 pad 7: /D9 -> /D10_SS
- J2 pad 8: /D8 -> /D9
- R2 pad 2: Net-(C4-Pad2) -> /RST
- SW1 pad 1: Net-(C4-Pad2) -> /RST
- U1 pad 29: Net-(C4-Pad2) -> /RST
Routing:
- net /RST: track 0.00 -> 76.9 mm
- net Net-(C4-Pad2): track 76.3 -> 0.00 mm
- net /VCC: track 179.1 -> 184.5 mm
- net GND: track 64.2 -> 62.6 mm
- net Net-(D4-Pad1): track 3.23 -> 2.10 mm
- net /D5: track 26.6 -> 25.9 mm

Commit message: UPDATE
Parts:
- added J5: AVR-ISP-6, Connector_PinHeader_2.54mm:PinHeader_2x03_P2.54mm_Vertical, F.Cu at (69.3, 64.9)
Routing:
- net /D11_MOSI: track 17.9 -> 40.6 mm, vias 0 -> 1
- net /D12_MISO: track 17.2 -> 36.2 mm, vias 0 -> 1
- net GND: track 62.6 -> 80.0 mm
- net /D13_SCK: track 46.3 -> 59.9 mm, vias 0 -> 1
- net /RST: track 76.9 -> 81.2 mm
- net /VCC: track 184.5 -> 187.5 mm
- net /D7: track 26.7 -> 27.4 mm
Other:
- board text added: "CTS"
- board text added: "D2"
- board text added: "D3"
- board text added: "D4"
- board text added: "D5"
- board text added: "D6"
- board text added: "D7"
- board text added: "DTR"
- board text added: "RX"
- board text added: "TX"
