File: Simpino_bareminimum/Simpino_bareminimum - Copy.kicad_pcb (KiCad board)
At the start: 2 copper layers, 50 x 49.8 mm, 22 parts, among them J1 North Junction, J2 South Junction, J3 West Junction, J4 East Junction, J5 AVR-ISP-6, SW1 SW_Push, U1 ATmega328P-AU, Y1 16mhz

Commit message: Update with diagrams
Other:
- net class Default: clearance 0.16 -> 0.2; trace_width 0.32 -> 0.35
- rule trace_clearance: 0.16 -> 0.2
Changed lines of the file:
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@@
   )
   (setup
-    (last_trace_width 0.32)
-    (trace_clearance 0.16)
+    (last_trace_width 0.35)
+    (trace_clearance 0.2)
     (zone_clearance 0.508)
     (zone_45_only no)
@@
     (mod_text_size 1 1)
     (mod_text_width 0.15)
-    (pad_size 1.524 1.524)
-    (pad_drill 0.762)
+    (pad_size 1.7 1.7)
+    (pad_drill 0)
     (pad_to_mask_clearance 0.05)
     (aux_axis_origin 0 0)
@@
   (net 30 /RST)
   (net_class Default "This is the default net class."
-    (clearance 0.16)
-    (trace_width 0.32)
+    (clearance 0.2)
+    (trace_width 0.35)
     (via_dia 0.8)
     (via_drill 0.4)
@@
       (effects (font (size 1.27 1.27) (thickness 0.15)))
     )
+    (fp_text user "West Junction" (at 69.915 64.6446 -180) (layer F.Fab)
+      (effects (font (size 1 1) (thickness 0.15)))
+    )
   )
